File: CST-104-DAS_Mother_Reverse/CST-104-DAS_Mother_Reverse.kicad_pcb (KiCad board)
At the start: 2 copper layers, 426 x 128 mm, 210 parts, among them J1 Conn_02x13_Odd_Even, J2 kailh-hotswap, K1 kailh-hotswap, M1 kailh-hotswap, P1 kailh-hotswap, Q1 kailh-hotswap, T1 kailh-hotswap, U1 kailh-hotswap, X1 kailh-hotswap, Y1 kailh-hotswap

Commit message: revision 0.1 is oredered!
update:
 - sch is updated
 - pcb is updated and traced
 - fabrical output is created and sent to production
 (ETA: 1 month)
Parts:
- removed TAB1: kailh-hotswap, switch:SW_Hotswap_Kailh_MX
- added ?: , , F.Cu at (132.5, 223.8)
- added ?: , , F.Cu at (109.5, 233.0)
- added ?: , , F.Cu at (456.5, 185.5)
- added ?: , , F.Cu at (249.0, 251.8)
- added ?: , , F.Cu at (342.0, 185.2)
- added ?: , , F.Cu at (327.8, 214.5)
- added ?: , , F.Cu at (394.8, 223.2)
- added ?: , , F.Cu at (394.5, 187.0)
- added ?: , , F.Cu at (86.0, 233.5)
- added ?: , , F.Cu at (267.2, 224.0)
- added ?: , , F.Cu at (265.8, 186.0)
- added ?: , , F.Cu at (498.0, 190.5)
- added ?: , , F.Cu at (133.2, 204.8)
- added ?: , , F.Cu at (180.5, 186.2)
- added ?: , , F.Cu at (457.0, 224.0)
- added ?: , , F.Cu at (294.0, 163.0)
- added ?: , , F.Cu at (346.2, 224.0)
- added ?: , , F.Cu at (178.8, 223.8)
- added ?: , , F.Cu at (348.5, 204.2)
- added G1: LOGO, LOGO, B.Cu at (367.0, 217.8)
- added G2: LOGO, LOGO, F.Cu at (415.2, 217.5)
- D1: renamed from D76; moved to B.Cu
- D10: renamed from D59; moved to B.Cu
- D100: renamed from D22; moved to B.Cu
- D101: renamed from D5; moved to B.Cu
- D102: renamed from D34; moved to B.Cu
- D103: renamed from D21; moved to B.Cu
- D104: renamed from D23; moved to B.Cu
- D105: renamed from D37; moved to B.Cu
- D11: renamed from D17; moved to B.Cu
- D12: renamed from D74; moved to B.Cu
- D13: renamed from D9; moved to B.Cu
- D14: renamed from D87; moved to B.Cu
- D15: renamed from D58; moved to B.Cu
- D16: renamed from D15; moved to B.Cu
- D17: renamed from D73; moved to B.Cu
- D18: renamed from D31; moved to B.Cu
- D19: renamed from D1; moved to B.Cu
- D2: renamed from D102; moved to B.Cu
- D20: renamed from D101; moved to B.Cu
- D21: renamed from D30; moved to B.Cu
- D22: renamed from D103; moved to B.Cu
- D23: renamed from D8; moved to B.Cu
- D24: renamed from D100; moved to B.Cu
- D25: renamed from D57; moved to B.Cu
- D26: renamed from D29; moved to B.Cu
- D27: renamed from D104; moved to B.Cu
- D28: renamed from D99; moved to B.Cu
- D29: renamed from D56; moved to B.Cu
- D3: renamed from D61; moved to B.Cu
- D30: renamed from D72; moved to B.Cu
- D31: renamed from D48; moved to B.Cu
- D32: renamed from D14; moved to B.Cu
- D33: renamed from D85; moved to B.Cu
- D34: renamed from D71; moved to B.Cu
- D35: renamed from D28; moved to B.Cu
- D36: renamed from D13; moved to B.Cu
- D37: renamed from D84; moved to B.Cu
- D38: renamed from D94; moved to B.Cu
- D39: renamed from D3; moved to B.Cu
- D4: renamed from D88; moved to B.Cu
- D40: renamed from D27; moved to B.Cu
- D41: renamed from D12; moved to B.Cu
- D42: renamed from D7; moved to B.Cu
- D43: renamed from D98; moved to B.Cu
- D44: renamed from D97; moved to B.Cu
- D45: renamed from D47; moved to B.Cu
- D46, J1: moved to B.Cu
- D47: renamed from D54; moved to B.Cu
- D48: renamed from D69; moved to B.Cu
- D49: renamed from D26; moved to B.Cu
- D5: renamed from D60; moved to B.Cu
- D50: renamed from D70; moved to B.Cu
- D51: renamed from D45; moved to B.Cu
- D52: renamed from D55; moved to B.Cu
- D53: renamed from D68; moved to B.Cu
- D54: renamed from D83; moved to B.Cu
- D55: renamed from D25; moved to B.Cu
- D56: renamed from D44; moved to B.Cu
- D57: renamed from D96; moved to B.Cu
- D58: renamed from D67; moved to B.Cu
- D59: renamed from D82; moved to B.Cu
- D6: renamed from D75; moved to B.Cu
- D60: renamed from D95; moved to B.Cu
- D61: renamed from D11; moved to B.Cu
- D62: renamed from D43; moved to B.Cu
- D63: renamed from D53; moved to B.Cu
- D64: renamed from D66; moved to B.Cu
- D65: renamed from D81; moved to B.Cu
- D66: renamed from D2; moved to B.Cu
- D67: renamed from D32; moved to B.Cu
- D68: renamed from D18; moved to B.Cu
- D69: renamed from D91; moved to B.Cu
- D7: renamed from D16; moved to B.Cu
- D70: renamed from D93; moved to B.Cu
- D71: renamed from D42; moved to B.Cu
- D72: renamed from D90; moved to B.Cu
- D73: renamed from D33; moved to B.Cu
- D74: renamed from D19; moved to B.Cu
- D75: renamed from D6; moved to B.Cu
- D76: renamed from D92; moved to B.Cu
- D77: renamed from D4; moved to B.Cu
- D78: renamed from D41; moved to B.Cu
- D79: renamed from D52; moved to B.Cu
- D8: renamed from D10; moved to B.Cu
- D80: renamed from D65; moved to B.Cu
- D81: renamed from D80; moved to B.Cu
- D83: renamed from D40; moved to B.Cu
- D84: renamed from D50; moved to B.Cu
- D85: renamed from D64; moved to B.Cu
- D86: renamed from D79; moved to B.Cu
- D87: renamed from D20; moved to B.Cu
- D88: renamed from D89; moved to B.Cu
- D89: renamed from D36; moved to B.Cu
- D9: renamed from D86; moved to B.Cu
- D90: renamed from D39; moved to B.Cu
- D91: renamed from D51; moved to B.Cu
- D92: renamed from D63; moved to B.Cu
- D93: renamed from D78; moved to B.Cu
- D94: renamed from D35; moved to B.Cu
- D95: renamed from D38; moved to B.Cu
- D96: renamed from D49; moved to B.Cu
- D97: renamed from D62; moved to B.Cu
- D98: renamed from D77; moved to B.Cu
- D99: renamed from D24; moved to B.Cu
- K1: renamed from Enter1; value kailh-hotswap -> Enter
- K10: renamed from RIgth1; value kailh-hotswap -> Rigth
- K100: renamed from V1; value kailh-hotswap -> V
- K101: renamed from C1; value kailh-hotswap -> C
- K102: renamed from X1; value kailh-hotswap -> X
- K103: renamed from Z1; value kailh-hotswap -> Z
- K104: renamed from Shift_L1; value kailh-hotswap -> Shift_L
- K11: renamed from Up1; value kailh-hotswap -> Up
- K12: renamed from 3_P1; value kailh-hotswap -> 3_P
- K13: renamed from 2_P1; value kailh-hotswap -> 2_P
- K14: renamed from 1_P1; value kailh-hotswap -> 1_P
- K15: renamed from 9_P1; value kailh-hotswap -> 9_P
- K16: renamed from 6_P1; value kailh-hotswap -> 6_P
- K17: renamed from 8_P1; value kailh-hotswap -> 8_P
- K18: renamed from 5_P1; value kailh-hotswap -> 5_P
- K19: renamed from 7_P1; value kailh-hotswap -> 7_P
- K2: renamed from Enter_P1; value kailh-hotswap -> Enter_P
- K20: renamed from 4_P1; value kailh-hotswap -> 4_P
- K21: renamed from -_P1; value kailh-hotswap -> -_P
- K22: renamed from +_P1; value kailh-hotswap -> +_P
- K23: renamed from *_P1; value kailh-hotswap -> *_P
- K24: renamed from /1; value kailh-hotswap -> /
- K25: renamed from Num1; value kailh-hotswap -> Num
- K26: renamed from PageUp1; value kailh-hotswap -> PageUp
- K27: renamed from PageDown1; value kailh-hotswap -> PageDown
- K28: renamed from Home1; value kailh-hotswap -> Home
- K29: renamed from End1; value kailh-hotswap -> End
- K3: renamed from Alt_L1; value kailh-hotswap -> Alt_L
- K30: renamed from Insert1; value kailh-hotswap -> Insert
- K31: renamed from Delete1; value kailh-hotswap -> Delete
- K32: renamed from Pause1; value kailh-hotswap -> Pause
- K33: renamed from Scroll1; value kailh-hotswap -> Scroll
- K34: renamed from SysIrq1; value kailh-hotswap -> SysIrq
- K35: renamed from F12; value kailh-hotswap -> F12
- K36: renamed from F11; value kailh-hotswap -> F11
- K37: renamed from F10; value kailh-hotswap -> F10
- K38: renamed from F9; value kailh-hotswap -> F9
- K39: renamed from F8; value kailh-hotswap -> F8
- K4: renamed from Win_L1; value kailh-hotswap -> Win_L
- K40: renamed from F7; value kailh-hotswap -> F7
- K41: renamed from F6; value kailh-hotswap -> F6
- K42: renamed from F5; value kailh-hotswap -> F5
- K43: renamed from F4; value kailh-hotswap -> F4
- K44: renamed from F3; value kailh-hotswap -> F3
- K45: renamed from F2; value kailh-hotswap -> F2
- K46: renamed from F1; value kailh-hotswap -> F1
- K47: renamed from ESC1; value kailh-hotswap -> ESC
- K48: renamed from BKSpc1; value kailh-hotswap -> BKSpc
- K49: renamed from =+1; value kailh-hotswap -> =+
- K5: renamed from Ctrl_l1; value kailh-hotswap -> Ctrl_l
- K50: renamed from -_1; value kailh-hotswap -> -_
- K51: renamed from _0; value kailh-hotswap -> 0
- K52: renamed from _9; value kailh-hotswap -> 9
- K53: renamed from _8; value kailh-hotswap -> 8
- K54: renamed from _7; value kailh-hotswap -> 7
- K55: renamed from _6; value kailh-hotswap -> 6
- K56: renamed from _5; value kailh-hotswap -> 5
- K57: renamed from _4; value kailh-hotswap -> 4
- K58: renamed from _3; value kailh-hotswap -> 3
- K59: renamed from _2; value kailh-hotswap -> 2
- K6: renamed from ._P1; value kailh-hotswap -> ._P
- K60: renamed from _1; value kailh-hotswap -> 1
- K61: renamed from "~"1; value kailh-hotswap -> "~"
- K62: renamed from \|1; value kailh-hotswap -> \|
- K63: renamed from ]}1; value kailh-hotswap -> ]}
- K64: renamed from [{1; value kailh-hotswap -> [{
- K65: renamed from P1; value kailh-hotswap -> P
- K66: renamed from O1; value kailh-hotswap -> O
- K67: renamed from I1; value kailh-hotswap -> I
- K68: renamed from U1; value kailh-hotswap -> U
- K69: renamed from Y1; value kailh-hotswap -> Y
- K7: renamed from 0_P1; value kailh-hotswap -> 0_P
- K70: renamed from T1; value kailh-hotswap -> T
- K71: renamed from R1; value kailh-hotswap -> R
- K72: renamed from E1; value kailh-hotswap -> E
- K73: renamed from W1; value kailh-hotswap -> W
- K74: renamed from Q1; value kailh-hotswap -> Q
- K75: renamed from TAB2; value kailh-hotswap -> TAB
- K76: renamed from ""1; value kailh-hotswap -> ""
- K77: renamed from ;:1; value kailh-hotswap -> ;:
- K78: renamed from L1; value kailh-hotswap -> L
- K79: renamed from K1; value kailh-hotswap -> K
- K8: renamed from Left1; value kailh-hotswap -> Left
- K80: renamed from J2; value kailh-hotswap -> J
- K81: renamed from H1; value kailh-hotswap -> H
- K82: renamed from G1; value kailh-hotswap -> G
- K83: renamed from F13; value kailh-hotswap -> F
- K84: renamed from D105; value kailh-hotswap -> D
- K85: renamed from S1; value kailh-hotswap -> S
- K86: renamed from A1; value kailh-hotswap -> A
- K87: renamed from CapsLock1; value kailh-hotswap -> CapsLock
- K88: renamed from Ctrl_R1; value kailh-hotswap -> Ctrl_R
- K89: renamed from Shift_R1; value kailh-hotswap -> Shift_R
- K9: renamed from Down1; value kailh-hotswap -> Down
- K90: renamed from /2; value kailh-hotswap -> /
- K91: renamed from APPS1; value kailh-hotswap -> APPS
- K92: renamed from Win_R1; value kailh-hotswap -> Win_R
- K93: renamed from >1; value kailh-hotswap -> >
- K94: renamed from <1; value kailh-hotswap -> <
- K95: renamed from Alt_R1; value kailh-hotswap -> Alt_R
- K96: renamed from M1; value kailh-hotswap -> M
- K97: renamed from N1; value kailh-hotswap -> N
- K98: renamed from Space1; value kailh-hotswap -> Space
- K99: renamed from B1; value kailh-hotswap -> B
- moved D105 351.0 mm to (91.9, 242.7), turned to 180 degrees
- moved D98 338.4 mm to (124.8, 223.8), turned to 180 degrees
- moved D97 324.3 mm to (123.2, 205.2), turned to 180 degrees
- moved D104 322.2 mm to (104.8, 222.6)
- moved D100 321.9 mm to (97.1, 205.3)
- moved D99 320.0 mm to (117.2, 241.0), turned to 90 degrees
- moved D102 318.1 mm to (93.8, 166.4)
- moved D103 315.7 mm to (95.9, 186.0)
- moved D93 315.1 mm to (151.1, 224.2), turned to 180 degrees
- moved D88 311.3 mm to (146.2, 247.2)
- moved D96 310.8 mm to (117.8, 186.5)
- moved D92 309.2 mm to (138.9, 205.3), turned to 180 degrees
- moved K12 301.1 mm to (475.5, 233.2)
- moved D86 297.8 mm to (170.2, 224.2), turned to 180 degrees
- moved D95 296.4 mm to (112.1, 167.3)
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Connections:
- D23 pad 2: unconnected-(D8-A-Pad2) -> /__11
- D31 pad 2: /__11 -> /__12
- K6 pad 1: unconnected-(._P1-Pad1) -> /__20
Routing:
- net /__11: track 0.00 -> 865.4 mm, vias 0 -> 15
- net /__18: track 0.00 -> 718.4 mm, vias 0 -> 11
- net /__16: track 0.00 -> 637.2 mm, vias 0 -> 13
- net /__12: track 0.00 -> 629.5 mm, vias 0 -> 13
- net /__9: track 0.00 -> 608.9 mm, vias 0 -> 6
- net /__17: track 0.00 -> 548.8 mm, vias 0 -> 17
- net /__7: track 0.00 -> 547.8 mm, vias 0 -> 3
- net /__8: track 0.00 -> 518.5 mm, vias 0 -> 2
- net /__22: track 0.00 -> 516.5 mm, vias 0 -> 12
- net /__24: track 0.00 -> 509.1 mm, vias 0 -> 3
- net /__19: track 0.00 -> 500.3 mm, vias 0 -> 16
- net /__21: track 0.00 -> 497.0 mm, vias 0 -> 14
- net /__25: track 0.00 -> 494.7 mm, vias 0 -> 4
- net /__5: track 0.00 -> 471.0 mm, vias 0 -> 2
- net /__2: track 0.00 -> 468.8 mm, vias 0 -> 6
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Other:
- outline, holes or cut-outs redrawn
- board text added: "1"
- board text added: "2"
- board text added: "25"
- board text added: "26"
- board text added: "CST-104-DAS_Mother PCB ver 4.0 06.05.2024 reverse rev. 0.1"
- board text added: "https://github.com/iarischenko/DasKeyboard_ReverseEngineering"
