File: CST-104-DAS_Mother_Reverse/CST-104-DAS_Mother_Reverse.kicad_sch (KiCad schematic)
At the start: 210 parts, among them J1 Conn_02x13_Odd_Even, J2 kailh-hotswap, K1 kailh-hotswap, M1 kailh-hotswap, P1 kailh-hotswap, Q1 kailh-hotswap, T1 kailh-hotswap, U1 kailh-hotswap, X1 kailh-hotswap, Y1 kailh-hotswap

Commit message: revision 0.1 is oredered!
update:
 - sch is updated
 - pcb is updated and traced
 - fabrical output is created and sent to production
 (ETA: 1 month)
Parts:
- removed TAB1: kailh-hotswap, switch:SW_Hotswap_Kailh_MX, symbol Switch:SW_Push
- K1: renamed from Enter1; value kailh-hotswap -> Enter
- K10: renamed from RIgth1; value kailh-hotswap -> Rigth
- K100: renamed from V1; value kailh-hotswap -> V
- K101: renamed from C1; value kailh-hotswap -> C
- K102: renamed from X1; value kailh-hotswap -> X
- K103: renamed from Z1; value kailh-hotswap -> Z
- K104: renamed from Shift_L1; value kailh-hotswap -> Shift_L
- K11: renamed from Up1; value kailh-hotswap -> Up
- K12: renamed from 3_P1; value kailh-hotswap -> 3_P
- K13: renamed from 2_P1; value kailh-hotswap -> 2_P
- K14: renamed from 1_P1; value kailh-hotswap -> 1_P
- K15: renamed from 9_P1; value kailh-hotswap -> 9_P
- K16: renamed from 6_P1; value kailh-hotswap -> 6_P
- K17: renamed from 8_P1; value kailh-hotswap -> 8_P
- K18: renamed from 5_P1; value kailh-hotswap -> 5_P
- K19: renamed from 7_P1; value kailh-hotswap -> 7_P
- K2: renamed from Enter_P1; value kailh-hotswap -> Enter_P
- K20: renamed from 4_P1; value kailh-hotswap -> 4_P
- K21: renamed from -_P1; value kailh-hotswap -> -_P
- K22: renamed from +_P1; value kailh-hotswap -> +_P
- K23: renamed from *_P1; value kailh-hotswap -> *_P
- K24: renamed from /1; value kailh-hotswap -> /
- K25: renamed from Num1; value kailh-hotswap -> Num
- K26: renamed from PageUp1; value kailh-hotswap -> PageUp
- K27: renamed from PageDown1; value kailh-hotswap -> PageDown
- K28: renamed from Home1; value kailh-hotswap -> Home
- K29: renamed from End1; value kailh-hotswap -> End
- K3: renamed from Alt_L1; value kailh-hotswap -> Alt_L
- K30: renamed from Insert1; value kailh-hotswap -> Insert
- K31: renamed from Delete1; value kailh-hotswap -> Delete
- K32: renamed from Pause1; value kailh-hotswap -> Pause
- K33: renamed from Scroll1; value kailh-hotswap -> Scroll
- K34: renamed from SysIrq1; value kailh-hotswap -> SysIrq
- K35: renamed from F12; value kailh-hotswap -> F12
- K36: renamed from F11; value kailh-hotswap -> F11
- K37: renamed from F10; value kailh-hotswap -> F10
- K38: renamed from F9; value kailh-hotswap -> F9
- K39: renamed from F8; value kailh-hotswap -> F8
- K4: renamed from Win_L1; value kailh-hotswap -> Win_L
- K40: renamed from F7; value kailh-hotswap -> F7
- K41: renamed from F6; value kailh-hotswap -> F6
- K42: renamed from F5; value kailh-hotswap -> F5
- K43: renamed from F4; value kailh-hotswap -> F4
- K44: renamed from F3; value kailh-hotswap -> F3
- K45: renamed from F2; value kailh-hotswap -> F2
- K46: renamed from F1; value kailh-hotswap -> F1
- K47: renamed from ESC1; value kailh-hotswap -> ESC
- K48: renamed from BKSpc1; value kailh-hotswap -> BKSpc
- K49: renamed from =+1; value kailh-hotswap -> =+
- K5: renamed from Ctrl_l1; value kailh-hotswap -> Ctrl_l
- K50: renamed from -_1; value kailh-hotswap -> -_
- K51: renamed from _0; value kailh-hotswap -> 0
- K52: renamed from _9; value kailh-hotswap -> 9
- K53: renamed from _8; value kailh-hotswap -> 8
- K54: renamed from _7; value kailh-hotswap -> 7
- K55: renamed from _6; value kailh-hotswap -> 6
- K56: renamed from _5; value kailh-hotswap -> 5
- K57: renamed from _4; value kailh-hotswap -> 4
- K58: renamed from _3; value kailh-hotswap -> 3
- K59: renamed from _2; value kailh-hotswap -> 2
- K6: renamed from ._P1; value kailh-hotswap -> ._P
- K60: renamed from _1; value kailh-hotswap -> 1
- K61: renamed from "~"1; value kailh-hotswap -> "~"
- K62: renamed from \|1; value kailh-hotswap -> \|
- K63: renamed from ]}1; value kailh-hotswap -> ]}
- K64: renamed from [{1; value kailh-hotswap -> [{
- K65: renamed from P1; value kailh-hotswap -> P
- K66: renamed from O1; value kailh-hotswap -> O
- K67: renamed from I1; value kailh-hotswap -> I
- K68: renamed from U1; value kailh-hotswap -> U
- K69: renamed from Y1; value kailh-hotswap -> Y
- K7: renamed from 0_P1; value kailh-hotswap -> 0_P
- K70: renamed from T1; value kailh-hotswap -> T
- K71: renamed from R1; value kailh-hotswap -> R
- K72: renamed from E1; value kailh-hotswap -> E
- K73: renamed from W1; value kailh-hotswap -> W
- K74: renamed from Q1; value kailh-hotswap -> Q
- K75: renamed from TAB2; value kailh-hotswap -> TAB
- K76: renamed from ""1; value kailh-hotswap -> ""
- K77: renamed from ;:1; value kailh-hotswap -> ;:
- K78: renamed from L1; value kailh-hotswap -> L
- K79: renamed from K1; value kailh-hotswap -> K
- K8: renamed from Left1; value kailh-hotswap -> Left
- K80: renamed from J2; value kailh-hotswap -> J
- K81: renamed from H1; value kailh-hotswap -> H
- K82: renamed from G1; value kailh-hotswap -> G
- K83: renamed from F13; value kailh-hotswap -> F
- K84: renamed from D105; value kailh-hotswap -> D
- K85: renamed from S1; value kailh-hotswap -> S
- K86: renamed from A1; value kailh-hotswap -> A
- K87: renamed from CapsLock1; value kailh-hotswap -> CapsLock
- K88: renamed from Ctrl_R1; value kailh-hotswap -> Ctrl_R
- K89: renamed from Shift_R1; value kailh-hotswap -> Shift_R
- K9: renamed from Down1; value kailh-hotswap -> Down
- K90: renamed from /2; value kailh-hotswap -> /
- K91: renamed from APPS1; value kailh-hotswap -> APPS
- K92: renamed from Win_R1; value kailh-hotswap -> Win_R
- K93: renamed from >1; value kailh-hotswap -> >
- K94: renamed from <1; value kailh-hotswap -> <
- K95: renamed from Alt_R1; value kailh-hotswap -> Alt_R
- K96: renamed from M1; value kailh-hotswap -> M
- K97: renamed from N1; value kailh-hotswap -> N
- K98: renamed from Space1; value kailh-hotswap -> Space
- K99: renamed from B1; value kailh-hotswap -> B
- renumbered D76 to D1, D59 to D10, D22 to D100, D5 to D101, D34 to D102, D21 to D103, D23 to D104, D37 to D105, D17 to D11, D74 to D12, D9 to D13, D87 to D14, D58 to D15, D15 to D16, D73 to D17, D31 to D18, D1 to D19, D102 to D2, D101 to D20, D30 to D21, D103 to D22, D8 to D23, D100 to D24, D57 to D25, D29 to D26, D104 to D27, D99 to D28, D56 to D29, D61 to D3, D72 to D30, D48 to D31, D14 to D32, D85 to D33, D71 to D34, D28 to D35, D13 to D36, D84 to D37, D94 to D38, D3 to D39, D88 to D4, D27 to D40, D12 to D41, D7 to D42, D98 to D43, D97 to D44, D47 to D45, D54 to D47, D69 to D48, D26 to D49, D60 to D5, D70 to D50, D45 to D51, D55 to D52, D68 to D53, D83 to D54, D25 to D55, D44 to D56, D96 to D57, D67 to D58, D82 to D59, D75 to D6, D95 to D60, D11 to D61, D43 to D62, D53 to D63, D66 to D64, D81 to D65, D2 to D66, D32 to D67, D18 to D68, D91 to D69, D16 to D7, D93 to D70, D42 to D71, D90 to D72, D33 to D73, D19 to D74, D6 to D75, D92 to D76, D4 to D77, D41 to D78, D52 to D79, D10 to D8, D65 to D80, D80 to D81, D40 to D83, D50 to D84, D64 to D85, D79 to D86, D20 to D87, D89 to D88, D36 to D89, D86 to D9, D39 to D90, D51 to D91, D63 to D92, D78 to D93, D35 to D94, D38 to D95, D49 to D96, D62 to D97, D77 to D98, D24 to D99
Connections:
- net __11: now also D23.2 (A); no longer D31.2 (A)
- net __12: now also D31.2 (A)
- net __20: now also K6.1
